Commit message: Enable Mode 99 SITL-based RL training and fix all launch bugs
- Add start_mode99_training.sh: runs arducopter binary directly (bypasses
  sim_vehicle.py/MAVProxy), polls TCP 5760 with nc -z, cleans up on exit
- Fix observation space: 25D → 26D (GPS is 4 elements, not 3)
- Add virtual obstacle simulation to ardupilot_gym_env.py: ray-AABB
  6-direction LiDAR matching physical RPi LiDAR format at flight time
- Fix connection ports: 5762 (MAVProxy) → 5760 (arducopter native)
- Remove EvalCallback and SubprocVecEnv from train_mode99_rl.py (MAVLink
  conflict; enforce n_envs=1)
- Fix scripts/start_sitl.sh: --load → --add-param-file, ARDUPILOT_DIR var
- Sync all physical model params to sysid_params.txt (mass=2.0, IXX=0.0347,
  IYY=0.0458, IZZ=0.0977, MAX_THRUST=8.0N, km=1.6e-7, TWR=1.6315)
- Update all documentation: RL_TRAINING_GUIDE, EXECUTION_GUIDE,
  MEDIUM_QUAD_MODEL, MODE99_OPERATION, README, SITL_TESTING_GUIDE

Co-Authored-By: Claude Sonnet 4.6 <noreply@anthropic.com>

File: drone_gym/assets/medium_quad.urdf (robot description, URDF)
Before this commit: robot medium_quad, 6 links, 5 joints
Links:
- link prop0_link: mass 0.05 -> 0.0
- link prop1_link: mass 0.05 -> 0.0
- link prop2_link: mass 0.05 -> 0.0
- link prop3_link: mass 0.05 -> 0.0
